File: eagle/namcogunpcb.brd (EAGLE design)
At the start: 88.9 x 25.4 mm, 23 parts, among them Q1 IRF530, Q2 BC337, Q3 BC337

Commit message: adding pcb as manufactured
Parts:
- removed AUDIO, GND, INDICATOR, SENSOR, TP1, TP2, TP3, TRIGGER, VCC: TPTP20SQ, testpad:TP20SQ
- removed JP4, JP5: (no value), pinhead:1X01
- added JP6: (no value), adafruit:1X03
- added JP8: (no value), pinhead:1X10
- added SV1: (no value), con-lstb:MA04-1
- added SV2: (no value), con-lstb:MA03-1
- D2: value (none) -> 1N4148DO35-7; device diode:DO35-10 -> diode:DO35-7
- JP3: device pinhead:1X01 -> pinhead:1X02
- JP7: device pinhead:1X10 -> pinhead:1X02
- R1: device resistor:0207/5V -> resistor:0207/10
- moved JP3 88.0 mm to (71.1, 17.8), turned to 180 degrees
- moved JP7 81.7 mm to (7.62, 17.8), turned to 0 degrees
- moved Q1 75.2 mm to (2.54, 7.62)
- moved R1 75.2 mm to (33.0, 8.26), turned to 180 degrees
- moved D2 73.8 mm to (31.8, 2.54), turned to 180 degrees
- moved D1 70.1 mm to (31.8, 5.08), turned to 180 degrees
- moved Q2 65.5 mm to (25.4, 13.3), turned to 180 degrees
- moved R2 62.9 mm to (33.0, 10.8), turned to 180 degrees
- moved JP2 62.9 mm to (74.9, 14.0)
- moved JP1 62.9 mm to (74.9, 11.4)
- moved R3 62.0 mm to (62.2, 12.7), turned to 180 degrees
- moved Q3 61.4 mm to (71.1, 12.7), turned to 90 degrees
Connections:
- net !POWERON: now also JP8.7; no longer JP7.9
- net !RELOAD-IN: now also JP8.2; no longer JP7.3
- net !TRIGGER: now also JP7.2, JP8.10; no longer JP7.1, TRIGGER.TP
- net 5V: now also JP6.1, JP8.4, SV1.1, SV2.1; no longer JP4.1, JP7.5, TP2.TP
- net AUDIO: now also JP6.2, JP8.1; no longer AUDIO.TP, JP7.2
- net GND: now also JP3.1, JP6.3, JP7.1, JP8.5, SV1.4, SV2.2; no longer GND.TP, JP5.1, JP7.6, TP3.TP
- net INDICATOR: now also JP8.8, SV1.2; no longer INDICATOR.TP, JP7.8
- net IRENABLE: now also JP8.3; no longer JP7.4
- net RELOAD-BUTT: now also JP3.2; no longer JP7.7, TP1.TP
- net SENSOR: now also JP8.9, SV1.3; no longer JP7.10, SENSOR.TP
- net VBATT: no longer VCC.TP
- net VSWITCHED: now also SV2.3; no longer JP3.1
Routing:
- net GND: track 100.2 -> 0.00 mm, vias 1 -> 0
- net 5V: track 30.5 -> 95.4 mm
- net !POWERON: track 68.6 -> 5.34 mm
- net SENSOR: track 61.0 -> 21.4 mm
- net RELOAD-BUTT: track 86.4 -> 47.3 mm
- net INDICATOR: track 61.0 -> 24.3 mm
- net N$2: track 15.2 -> 43.8 mm
- net !TRIGGER: track 61.0 -> 34.3 mm
- net AUDIO: track 22.9 -> 9.42 mm
- net VBATT: track 15.2 -> 23.6 mm
- net !RELOAD-IN: track 30.5 -> 35.3 mm
- net N$3: track 5.08 -> 1.91 mm
- net N$4: track 0.00 -> 2.80 mm
- net IRENABLE: track 7.62 -> 9.42 mm
- added copper zone on layer 1, net GND
- added copper zone on layer 16, net GND
Other:
- board size 88.9 x 25.4 mm -> 87 x 25.4 mm
- board text added: "audio"
- board text added: "boost"
- board text added: "ir led"
- board text added: "reload"
- board text added: "sensor"
- board text added: "trig"
- board text removed: "X"
- board text removed: "don't forget to jumper around the cuts in tracks 1 & 10"
- board text removed: "from VOUT+ on boost board"
- board text removed: "to VIN+ on boost board"
- board text removed: "to VIN- on boost board"
