File: eagle/namcogunpcb.sch (EAGLE design)
At the start: 23 parts, among them Q1 IRF530, Q2 BC337, Q3 BC337

Commit message: adding pcb as manufactured
Parts:
- removed AUDIO, GND, INDICATOR, SENSOR, TP1, TP2, TP3, TRIGGER, VCC: TPTP20SQ, testpad:TPTP20SQ
- removed JP4, JP5: (no value), pinhead:PINHD-1X1
- added JP6: (no value), adafruit:PINHD-1X3
- added JP8: (no value), pinhead:PINHD-1X10
- added SV1: (no value), con-lstb:MA04-1
- added SV2: (no value), con-lstb:MA03-1
- D2: value (none) -> 1N4148DO35-7; device diode:DIODE-DO35-10 -> diode:1N4148DO35-7
- JP3: device pinhead:PINHD-1X1 -> pinhead:PINHD-1X2
- JP7: device pinhead:PINHD-1X10 -> pinhead:PINHD-1X2
- R1: device resistor:R-EU_0207/5V -> resistor:R-EU_0207/10
Connections:
- net !POWERON: now also JP8.7; no longer JP7.9
- net !RELOAD-IN: now also JP8.2; no longer JP7.3
- net !TRIGGER: now also JP7.2, JP8.10; no longer JP7.1, TRIGGER.TP
- net 5V: now also JP6.1, JP8.4, SV1.1, SV2.1; no longer JP4.1, JP7.5, TP2.TP
- net AUDIO: now also JP6.2, JP8.1; no longer AUDIO.TP, JP7.2
- net GND: now also JP3.1, JP6.3, JP7.1, JP8.5, SV1.4, SV2.2; no longer GND.TP, JP5.1, JP7.6, TP3.TP
- net INDICATOR: now also JP8.8, SV1.2; no longer INDICATOR.TP, JP7.8
- net IRENABLE: now also JP8.3; no longer JP7.4
- net RELOAD-BUTT: now also JP3.2; no longer JP7.7, TP1.TP
- net SENSOR: now also JP8.9, SV1.3; no longer JP7.10, SENSOR.TP
- net VBATT: no longer VCC.TP
- net VSWITCHED: now also SV2.3; no longer JP3.1
Other:
- moved on the sheet: D1, D2, JP1, JP2, Q1, Q2, Q3, R1, R2, R3
